File: Example/Example.sch (EAGLE design)
At the start: 11 parts, among them IC1 LM555D, J1 UX60-MB-5S8, Q2 BSS806N, SW1 MFS101D-6-Z

Commit message: Delete motor
commit test
Parts:
- removed JP1: (no value), RoboJackets-Connectors:PINHD-1X2
- removed Q2: BSS806N, RoboJackets-Discrete:BSS806N
Connections:
- removed net N$2: JP1.2, Q2.D
- net +9V: no longer JP1.1
- net GND: no longer Q2.S
- net T_OUT: no longer Q2.G
Other:
- note removed: "Low side switch using 2.3A rated transistor and 450mA max current motor"
- note removed: "Motor"
- note removed: "Motor externally wired to this plug"
Changed lines of the file:
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@@
 <?xml version="1.0" encoding="utf-8"?>
 <!DOCTYPE eagle SYSTEM "eagle.dtd">
-<eagle version="9.5.2">
+<eagle version="9.5.1">
 <drawing>
 <settings>
@@
 <part name="SUPPLY5" library="RoboJackets-Supplies" deviceset="GND" device=""/>
 <part name="C3" library="rcl" library_urn="urn:adsk.eagle:library:334" deviceset="C-US" device="C0603" package3d_urn="urn:adsk.eagle:package:23616/2" value="0.01uF"/>
-<part name="Q2" library="RoboJackets-Discrete" deviceset="BSS806N" device="" override_package3d_urn="urn:adsk.eagle:package:25000917/2" override_package_urn="urn:adsk.eagle:footprint:25000918/1"/>
-<part name="SUPPLY6" library="RoboJackets-Supplies" deviceset="GND" device=""/>
 <part name="J2" library="RoboJackets-Connectors" deviceset="PJ-037A*" device="" override_package3d_urn="urn:adsk.eagle:package:25000921/2" override_package_urn="urn:adsk.eagle:footprint:25000922/1"/>
-<part name="JP1" library="RoboJackets-Connectors" deviceset="PINHD-1X2" device="" package3d_urn="urn:adsk.eagle:package:22435/2"/>
-<part name="SUPPLY7" library="RoboJackets-Supplies" deviceset="+9V" device=""/>
 <part name="SUPPLY8" library="RoboJackets-Supplies" deviceset="GND" device=""/>
 <part name="SUPPLY9" library="RoboJackets-Supplies" deviceset="+9V" device=""/>
@@
 Both are within operating voltage of motor and outside
 of audio range. </text>
-<text x="182.88" y="172.72" size="1.778" layer="97">Motor externally wired to this plug</text>
-<text x="182.88" y="134.62" size="1.778" layer="97">Low side switch using 2.3A rated
-transistor and 450mA max current
-motor</text>
 <text x="25.4" y="139.7" size="1.778" layer="97">USB or Barrel Jack power (5-9V)</text>
 <wire x1="15.24" y1="127" x2="137.16" y2="127" width="0.1524" layer="97" style="shortdash"/>
@@
 <wire x1="228.6" y1="195.58" x2="144.78" y2="195.58" width="0.1524" layer="97" style="shortdash"/>
 <wire x1="144.78" y1="195.58" x2="144.78" y2="127" width="0.1524" layer="97" style="shortdash"/>
-<text x="154.94" y="187.96" size="1.778" layer="97">Motor</text>
 </plain>
 <instances>
@@
 <attribute name="VALUE" x="28.956" y="66.929" size="1.778" layer="96"/>
 </instance>
-<instance part="Q2" gate="G$1" x="172.72" y="149.86" smashed="yes">
-<attribute name="VALUE" x="175.26" y="147.32" size="1.778" layer="96"/>
-<attribute name="NAME" x="175.26" y="152.4" size="1.778" layer="95"/>
-</instance>
-<instance part="SUPPLY6" gate="G$1" x="172.72" y="137.16" smashed="yes">
-<attribute name="VALUE" x="170.18" y="134.62" size="1.778" layer="96"/>
-</instance>
 <instance part="J2" gate="G$1" x="35.56" y="149.86" smashed="yes">
 <attribute name="NAME" x="25.4" y="157.48" size="1.778" layer="95"/>
 <attribute name="VALUE" x="25.4" y="144.78" size="1.778" layer="96"/>
-</instance>
-<instance part="JP1" gate="G$1" x="182.88" y="165.1" smashed="yes">
-<attribute name="NAME" x="176.53" y="170.815" size="1.778" layer="95"/>
-<attribute name="VALUE" x="176.53" y="160.02" size="1.778" layer="96"/>
-</instance>
-<instance part="SUPPLY7" gate="+9V" x="172.72" y="177.8" smashed="yes">
-<attribute name="VALUE" x="170.815" y="180.975" size="1.778" layer="96"/>
 </instance>
 <instance part="SUPPLY8" gate="G$1" x="86.36" y="137.16" smashed="yes">
@@
 <pinref part="SUPPLY3" gate="G$1" pin="GND"/>
 <wire x1="81.28" y1="66.04" x2="81.28" y2="58.42" width="0.1524" layer="91"/>
-</segment>
-<segment>
-<pinref part="SUPPLY6" gate="G$1" pin="GND"/>
-<pinref part="Q2" gate="G$1" pin="S"/>
-<wire x1="172.72" y1="139.7" x2="172.72" y2="144.78" width="0.1524" layer="91"/>
 </segment>
 <segment>
@@
 </segment>
 <segment>
-<pinref part="JP1" gate="G$1" pin="1"/>
-<wire x1="180.34" y1="167.64" x2="172.72" y2="167.64" width="0.1524" layer="91"/>
-<wire x1="172.72" y1="167.64" x2="172.72" y2="175.26" width="0.1524" layer="91"/>
-<pinref part="SUPPLY7" gate="+9V" pin="+9V"/>
-</segment>
-<segment>
 <pinref part="SUPPLY9" gate="+9V" pin="+9V"/>
 <wire x1="124.46" y1="157.48" x2="124.46" y2="162.56" width="0.1524" layer="91"/>
@@
 <label x="60.96" y="86.36" size="1.27" layer="95" xref="yes"/>
 </segment>
-<segment>
-<pinref part="Q2" gate="G$1" pin="G"/>
-<wire x1="167.64" y1="147.32" x2="162.56" y2="147.32" width="0.1524" layer="91"/>
-<label x="162.56" y="147.32" size="1.27" layer="95" rot="R180" xref="yes"/>
-</segment>
 </net>
 <net name="N$1" class="0">
@@
 </segment>
 </net>
-<net name="N$2" class="0">
-<segment>
-<pinref part="JP1" gate="G$1" pin="2"/>
-<pinref part="Q2" gate="G$1" pin="D"/>
-<wire x1="180.34" y1="165.1" x2="172.72" y2="165.1" width="0.1524" layer="91"/>
-<wire x1="172.72" y1="165.1" x2="172.72" y2="154.94" width="0.1524" layer="91"/>
-</segment>
-</net>

Commit message: Update Example.sch
Added labels to the schematic view of parts we need.
Other:
- note added: "Decade Counter"
- note added: "SR latch"
Changed lines of the file:
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@@
 <?xml version="1.0" encoding="utf-8"?>
 <!DOCTYPE eagle SYSTEM "eagle.dtd">
-<eagle version="9.5.1">
+<eagle version="9.5.2">
 <drawing>
 <settings>
@@
 <wire x1="228.6" y1="195.58" x2="144.78" y2="195.58" width="0.1524" layer="97" style="shortdash"/>
 <wire x1="144.78" y1="195.58" x2="144.78" y2="127" width="0.1524" layer="97" style="shortdash"/>
+<text x="124.46" y="114.3" size="1.778" layer="97">SR latch</text>
+<text x="172.72" y="114.3" size="1.778" layer="97">Decade Counter</text>
 </plain>
 <instances>
