File: Example/Example.brd (EAGLE design)
At the start: 86 x 54 mm, 12 parts, among them IC1 LM555D, J1 UX60-MB-5S8, Q2 BSS806N, SW1 MFS101D-6-Z

Commit message: Delete motor
commit test
Parts:
- removed JP1: (no value), RoboJackets-Connectors:1X02
- removed Q2: BSS806N, RoboJackets-Discrete:SOT-23-3
Connections:
- removed net N$2: JP1.2, Q2.3
- net +9V: no longer JP1.1
- net GND: no longer Q2.2
- net T_OUT: no longer Q2.1
Routing:
- net N$2: track 5.56 -> 0.00 mm
- net +9V: track 40.6 -> 37.0 mm
- net GND: track 13.5 -> 12.0 mm, vias 7 -> 6
Changed lines of the file:
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@@
 <?xml version="1.0" encoding="utf-8"?>
 <!DOCTYPE eagle SYSTEM "eagle.dtd">
-<eagle version="9.5.2">
+<eagle version="9.5.1">
 <drawing>
 <settings>
-<setting alwaysvectorfont="yes"/>
+<setting alwaysvectorfont="no"/>
 <setting verticaltext="up"/>
 </settings>
@@
 <attribute name="NAME" x="18.616" y="21.773" size="1.27" layer="25" font="vector" ratio="10" rot="R180"/>
 </element>
-<element name="Q2" library="RoboJackets-Discrete" package="SOT-23-3" override_package3d_urn="urn:adsk.eagle:package:25000917/2" override_package_urn="urn:adsk.eagle:footprint:25000918/1" value="BSS806N" x="8.37" y="19.36" smashed="yes" rot="R90">
-<attribute name="DKPN" value="BSS806NH6327XTSA1CT-ND" x="31.23" y="46.03" size="1.778" layer="27" rot="R90" display="off"/>
-<attribute name="NAME" x="9.37" y="17.36" size="1" layer="25" font="vector" rot="R180"/>
-</element>
 <element name="TM1" library="adafruit" library_urn="urn:adsk.eagle:library:420" package="TRIM-3386" package3d_urn="urn:adsk.eagle:package:6240934/1" value="" x="20.36" y="6.19" smashed="yes">
 <attribute name="NAME" x="15.28" y="4.115" size="1.27" layer="25" font="vector" rot="R90"/>
@@
 <attribute name="NAME" x="9.782" y="9.34" size="1" layer="25" font="vector"/>
 <attribute name="VALUE" x="-2.438" y="-0.46" size="1" layer="27" font="vector" align="top-left"/>
-</element>
-<element name="JP1" library="RoboJackets-Connectors" package="1X02" package3d_urn="urn:adsk.eagle:package:22435/2" value="" x="8.77" y="13.19" smashed="yes" rot="R90">
-<attribute name="NAME" x="11.1812" y="11.8438" size="1" layer="25" font="vector" rot="R90"/>
-<attribute name="POPULARITY" value="98" x="8.77" y="13.19" size="1.778" layer="27" rot="R90" display="off"/>
-<attribute name="VALUE" x="10.775" y="10.65" size="1" layer="27" font="vector" rot="R90" align="top-left"/>
 </element>
 <element name="U$2" library="RoboJackets-Aesthetics" package="ROBOBUZZ_1.4X" value="" x="39.25" y="2.36" smashed="yes"/>
@@
 <contactref element="C2" pad="2"/>
 <contactref element="C1" pad="2"/>
-<contactref element="Q2" pad="2"/>
 <contactref element="J2" pad="P$1"/>
 <contactref element="C3" pad="2"/>
-<wire x1="9.57" y1="20.31" x2="9.57" y2="21.17" width="0.4" layer="1"/>
-<wire x1="9.57" y1="21.17" x2="9.11" y2="21.63" width="0.4" layer="1"/>
-<via x="9.11" y="21.63" extent="1-16" drill="0.35"/>
 <wire x1="11.5" y1="23.43" x2="10.85" y2="24.08" width="0.2" layer="1"/>
 <wire x1="10.85" y1="24.08" x2="10.06" y2="24.08" width="0.2" layer="1"/>
@@
 <wire x1="15.877" y1="13.783" x2="16.17" y2="13.49" width="0.2" layer="1"/>
 <via x="16.17" y="13.49" extent="1-16" drill="0.35"/>
+<wire x1="10.06" y1="24.08" x2="9.58" y2="32.46" width="0" layer="19" extent="1-1"/>
+<wire x1="13.11" y1="24.29" x2="11.5" y2="23.43" width="0" layer="19" extent="1-1"/>
+<wire x1="20.2944" y1="15.719" x2="14.546" y2="23.495" width="0" layer="19" extent="1-1"/>
+<wire x1="16.17" y1="13.49" x2="20.2944" y2="15.719" width="0" layer="19" extent="1-1"/>
+<wire x1="14.105" y1="11.66" x2="14.105" y2="13.783" width="0" layer="19" extent="1-1"/>
+<wire x1="4.562" y1="4.54" x2="13.54" y2="9.9" width="0" layer="19" extent="1-1"/>
 </signal>
 <signal name="+9V">
@@
 <contactref element="IC1" pad="8"/>
 <contactref element="C2" pad="1"/>
-<contactref element="JP1" pad="1"/>
 <wire x1="14.1476" y1="15.719" x2="14.17" y2="15.6966" width="0.2" layer="1"/>
 <wire x1="20.2944" y1="19.529" x2="21.491" y2="19.529" width="0.2" layer="1"/>
@@
 <wire x1="4.8" y1="19.57" x2="5.45" y2="19.57" width="0.4" layer="1"/>
 <wire x1="6.44" y1="18.58" x2="6.44" y2="13.99" width="0.4" layer="1"/>
-<wire x1="8.77" y1="11.92" x2="8.51" y2="11.92" width="0.4" layer="1"/>
 <wire x1="8.51" y1="11.92" x2="6.44" y2="13.99" width="0.4" layer="1"/>
 <wire x1="14.1476" y1="15.719" x2="12.405" y2="13.9764" width="0.2" layer="1"/>
 <wire x1="12.405" y1="13.9764" x2="12.405" y2="13.783" width="0.4" layer="1"/>
 <wire x1="12.405" y1="13.783" x2="12.405" y2="11.66" width="0.2" layer="1"/>
-<wire x1="8.77" y1="11.92" x2="12.145" y2="11.92" width="0.4" layer="1"/>
 <wire x1="12.145" y1="11.92" x2="12.405" y2="11.66" width="0.4" layer="1"/>
 <wire x1="17.82" y1="3.3325" x2="12.405" y2="8.7475" width="0.2" layer="1"/>
 <wire x1="12.405" y1="8.7475" x2="12.405" y2="11.66" width="0.2" layer="1"/>
+<wire x1="12.145" y1="11.92" x2="8.51" y2="11.92" width="0" layer="19" extent="1-1"/>
 </signal>
 <signal name="THR">
@@
 <signal name="T_OUT">
 <contactref element="IC1" pad="3"/>
-<contactref element="Q2" pad="1"/>
 <wire x1="20.2944" y1="18.259" x2="18.601" y2="18.259" width="0.2" layer="1"/>
 <wire x1="18.601" y1="18.259" x2="18.6" y2="18.26" width="0.2" layer="1"/>
@@
 <via x="11.88" y="18.2" extent="1-16" drill="0.35"/>
 <wire x1="11.88" y1="18.2" x2="9.78" y2="18.2" width="0.2" layer="1"/>
-<wire x1="9.78" y1="18.2" x2="9.57" y2="18.41" width="0.2" layer="1"/>
 </signal>
 <signal name="N$1">
@@
 <wire x1="14.1476" y1="21.3966" x2="14.546" y2="21.795" width="0.2" layer="1"/>
 </signal>
-<signal name="N$2">
-<contactref element="JP1" pad="2"/>
-<contactref element="Q2" pad="3"/>
-<wire x1="7.17" y1="19.36" x2="8.77" y2="17.76" width="0.4" layer="1"/>
-<wire x1="8.77" y1="17.76" x2="8.77" y2="14.46" width="0.4" layer="1"/>
-</signal>
 <signal name="N$4">

Commit message: add
add parts
Parts:
- removed C1, C3: 0.01uF, rcl:C0603
- removed C2: 0.1uF, rcl:C0603
- removed C4: 10uF, rcl:C0603
- removed IC1: LM555D, adafruit:SO08
- removed J1: UX60-MB-5S8, RoboJackets-Connectors:UX60-MB-5S8
- removed J2: (no value), RoboJackets-Connectors:PJ-037A
- removed SW1: MFS101D-6-Z, Example:MFS101D-6-Z
- removed TM1: (no value), adafruit:TRIM-3386
- added R1: 330, RoboJackets-Resistors:GHOST_0.075
- added S1, S2: (no value), adafruit:B3F-40XX
- added U$1, U$3: (no value), adafruit:CR1220-SMD
Connections:
- removed net +9V: C2.1, C4.1, IC1.4, IC1.8, SW1.2, TM1.1
- removed net GND: C1.2, C2.2, C3.2, C4.2, IC1.1, J1.5, J2.P$1
- removed net N$1: IC1.7, TM1.2
- removed net N$3: C3.1, IC1.5
- removed net N$4: J1.1, SW1.3
- removed net N$6: J2.P$2, SW1.1
- removed net THR: C1.1, IC1.2, IC1.6, TM1.3
- removed net T_OUT: IC1.3
Routing:
- net +9V: track 37.0 -> 0.00 mm, vias 2 -> 0
- net THR: track 29.4 -> 0.00 mm
- net N$4: track 19.3 -> 0.00 mm
- net N$1: track 18.8 -> 0.00 mm
- net N$6: track 15.4 -> 0.00 mm
- net GND: track 12.0 -> 0.00 mm, vias 6 -> 0
- net T_OUT: track 10.5 -> 0.00 mm, vias 2 -> 0
- net N$3: track 2.43 -> 0.00 mm

Commit message: Revert "add"
This reverts commit c6e4ebc28e4f55c76fdda87922b953a09ff3b68b.
Parts:
- removed R1: 330, RoboJackets-Resistors:GHOST_0.075
- removed S1, S2: (no value), adafruit:B3F-40XX
- removed U$1, U$3: (no value), adafruit:CR1220-SMD
- added C1, C3: 0.01uF, rcl:C0603
- added C2: 0.1uF, rcl:C0603
- added C4: 10uF, rcl:C0603
- added IC1: LM555D, adafruit:SO08
- added J1: UX60-MB-5S8, RoboJackets-Connectors:UX60-MB-5S8
- added J2: (no value), RoboJackets-Connectors:PJ-037A
- added SW1: MFS101D-6-Z, Example:MFS101D-6-Z
- added TM1: (no value), adafruit:TRIM-3386
Connections:
- new net +9V: C2.1, C4.1, IC1.4, IC1.8, SW1.2, TM1.1
- new net GND: C1.2, C2.2, C3.2, C4.2, IC1.1, J1.5, J2.P$1
- new net N$1: IC1.7, TM1.2
- new net N$3: C3.1, IC1.5
- new net N$4: J1.1, SW1.3
- new net N$6: J2.P$2, SW1.1
- new net THR: C1.1, IC1.2, IC1.6, TM1.3
- new net T_OUT: IC1.3
Routing:
- net +9V: track 0.00 -> 37.0 mm, vias 0 -> 2
- net THR: track 0.00 -> 29.4 mm
- net N$4: track 0.00 -> 19.3 mm
- net N$1: track 0.00 -> 18.8 mm
- net N$6: track 0.00 -> 15.4 mm
- net GND: track 0.00 -> 12.0 mm, vias 0 -> 6
- net T_OUT: track 0.00 -> 10.5 mm, vias 0 -> 2
- net N$3: track 0.00 -> 2.43 mm
