File: Example/Example.brd (EAGLE design)
At the start: 86 x 54 mm, 29 parts, among them IC2 74LS02D, IC3 74LS02D, U1 CD4017

Commit message: moved stuff
move
Parts:
- moved U$4 239.2 mm to (74.1, 42.7)
- moved U$5 224.4 mm to (74.5, 11.6)
- moved S3 168.3 mm to (76.3, -21.8)
- moved U$3 129.2 mm to (14.9, 44.2)
- moved S2 106.1 mm to (-40.2, 46.5)
- moved D4 86.9 mm to (22.0, -31.4)
- moved D5 86.9 mm to (22.0, -35.7)
- moved D6 86.9 mm to (22.0, -40.0)
- moved R4 86.9 mm to (20.6, -70.2)
- moved R5 86.9 mm to (20.6, -75.1)
- moved R6 86.9 mm to (20.6, -95.3)
- moved D1 86.9 mm to (22.0, -27.1)
- moved D10 86.9 mm to (22.0, -57.1)
- moved D11 86.9 mm to (22.0, -61.4)
- moved D12 86.9 mm to (22.0, -65.6)
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Routing:
- removed copper zone on layer 16, net GND
Other:
- board text removed: "RoboJackets PCB Contest 555 Timer PWM Motor Driver"

Commit message: Revert "moved stuff"
This reverts commit 32ee3d4f72a0406771ac1d0ac5515acdafe1b475.
Parts:
- moved U$4 239.2 mm to (-21.4, -176.6)
- moved U$5 224.4 mm to (-21.4, -191.3)
- moved S3 168.3 mm to (-23.8, -157.1)
- moved U$3 129.2 mm to (-21.4, -79.8)
- moved S2 106.1 mm to (-23.8, -58.2)
- moved D4 86.9 mm to (-28.4, -102.2)
- moved D5 86.9 mm to (-28.4, -106.5)
- moved D6 86.9 mm to (-28.4, -110.8)
- moved R4 86.9 mm to (-29.8, -141.0)
- moved R5 86.9 mm to (-29.8, -145.9)
- moved R6 86.9 mm to (-29.8, -166.2)
- moved D1 86.9 mm to (-28.4, -98.0)
- moved D10 86.9 mm to (-28.4, -127.9)
- moved D11 86.9 mm to (-28.4, -132.2)
- moved D12 86.9 mm to (-28.4, -136.5)
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Routing:
- added copper zone on layer 16, net GND
Other:
- board text added: "RoboJackets PCB Contest 555 Timer PWM Motor Driver"
